File: kicad/limbcontroller/limbcontroller.kicad_sch (KiCad schematic)
At the start: 34 parts, among them J3 Screw_Terminal_01x05, J4 Screw_Terminal_01x05, J5 USB_C_Receptacle_USB2.0_14P, M1 Stepper_Motor_bipolar, Q1 DTB143EK, SW2 1825910-6, SW3 1825910-6, U1 RT9193-33GB, U5 STM32F103C8T6, U6 BMI323

Commit message: cleaned up kicad files and changed 1uf capacitors to 0805 SMD size
Parts:
- C2, C21: footprint Capacitor_SMD:C_01005_0402Metric_Pad0.57x0.30mm_HandSolder -> Capacitor_SMD:C_0805_2012Metric_Pad1.18x1.45mm_HandSolder
Changed lines of the file:
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@@
 			)
 		)
-		(property "Footprint" "Capacitor_SMD:C_01005_0402Metric_Pad0.57x0.30mm_HandSolder"
+		(property "Footprint" "Capacitor_SMD:C_0805_2012Metric_Pad1.18x1.45mm_HandSolder"
 			(at 195.2752 144.78 0)
 			(hide yes)
@@
 			)
 		)
-		(property "Footprint" "Capacitor_SMD:C_01005_0402Metric_Pad0.57x0.30mm_HandSolder"
+		(property "Footprint" "Capacitor_SMD:C_0805_2012Metric_Pad1.18x1.45mm_HandSolder"
 			(at 241.6048 146.05 0)
 			(hide yes)
