File: kicad/maincontroller/maincontroller.kicad_sch (KiCad schematic)
At the start: 19 parts, among them J1 XT60PW-M, J2 Screw_Terminal_01x05, U2 ESP32-S3-DEVKITC-1-N8R2, U3 LM2596S-3.3_NOPB, U4 LTC4311ISC6_TRPBF

Commit message: cleaned up kicad files and changed 1uf capacitors to 0805 SMD size
Parts:
- C14, C18: footprint Capacitor_SMD:C_01005_0402Metric_Pad0.57x0.30mm_HandSolder -> Capacitor_SMD:C_0805_2012Metric_Pad1.18x1.45mm_HandSolder
Changed lines of the file:
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@@
 			)
 		)
-		(property "Footprint" "Capacitor_SMD:C_01005_0402Metric_Pad0.57x0.30mm_HandSolder"
+		(property "Footprint" "Capacitor_SMD:C_0805_2012Metric_Pad1.18x1.45mm_HandSolder"
 			(at 147.0152 143.51 0)
 			(hide yes)
@@
 			)
 		)
-		(property "Footprint" "Capacitor_SMD:C_01005_0402Metric_Pad0.57x0.30mm_HandSolder"
+		(property "Footprint" "Capacitor_SMD:C_0805_2012Metric_Pad1.18x1.45mm_HandSolder"
 			(at 162.2552 143.51 0)
 			(hide yes)
